Commit message: Added camera to xacro files

File: config/arm.xacro (robot description, xacro)
@@ -67,3 +67,9 @@
     <xacro:configure_collisions link="6" />
     <xacro:configure_collisions link="7" />
+<!-- Disable some collision of camera with arm links  -->
+    <xacro:property name="link_camera" value="$(arg arm_id)_link{}" />
+    <xacro:disable_collisions_for link="fake_camera_link" others="${[link_camera.format(i) for i in python.range(5,8)]}" />
+    <!-- Disable collision of camera with _sc links -->
+    <xacro:property name="link_camera" value="$(arg arm_id)_link{}_sc" />
+    <xacro:disable_collisions_for link="fake_camera_link" others="${[link_camera.format(i) for i in python.range(5,8)]}" />
 </robot>

File: config/hand.xacro (robot description, xacro)
@@ -38,4 +38,9 @@
         <xacro:disable_collisions_for link="$(arg arm_id)_rightfinger" others="${list(others)}" />
         <disable_collisions link1="$(arg arm_id)_leftfinger" link2="$(arg arm_id)_rightfinger" reason="Never" />
+        <!-- DISABLE COLLISION FOR CAMERA AND HAND-->
+        <disable_collisions link1="fake_camera_link" link2="$(arg arm_id)_hand" reason="Never" />
+        <disable_collisions link1="fake_camera_link" link2="$(arg arm_id)_hand_sc" reason="Never" />
+        <disable_collisions link1="fake_camera_link" link2="$(arg arm_id)_rightfinger" reason="Never" />
+        <disable_collisions link1="fake_camera_link" link2="$(arg arm_id)_leftfinger" reason="Never" />
     </xacro:macro>
 </robot>

File: config/panda.srdf.xacro (robot description, xacro)
@@ -9,4 +9,5 @@
     <!-- panda_arm group: eef frame aligned to robot's flanche -->
     <xacro:arm name="$(arg arm_id)_arm" tip_link="$(arg arm_id)_link8"/>
+    <xacro:arm name="$(arg arm_id)_camera" tip_link="fake_camera_link"/>
     <!--Add the hand if people request it-->
     <xacro:arg name="hand" default="false" />
